File: Hardware/Port_temp_hw/pcb.brd (EAGLE design)
At the start: 76.2 x 62.2 mm, 6 parts

Commit message: hg
Parts:
- moved JP3 8.89 mm to (62.2, 27.9)
- moved JP1 6.35 mm to (49.5, 49.5)
- moved R1 3.81 mm to (53.3, 26.7)
- moved WIFI_CONN 1.80 mm to (12.7, 50.8)
Routing:
- net GND: track 230.7 -> 218.4 mm
- net VCC: track 23.2 -> 16.8 mm
- net N$7: track 8.89 -> 3.81 mm
- net N$8: track 6.35 -> 2.54 mm
- net WIFI_RX: track 20.0 -> 18.2 mm
- net 3V3: track 78.8 -> 77.6 mm
- net WIFI_CE: track 51.8 -> 51.1 mm
- net WIFI_RESET: track 45.7 -> 45.0 mm
- net WIFI_TX: track 44.0 -> 43.3 mm
Other:
- board size 76.2 x 62.2 mm -> 64.8 x 54.6 mm
